Commit message: Added a node which sets a sinusoidal position input, tried to tune the PIDs

File: camera/urdf/camera_gazebo.xacro (robot description, xacro)
@@ -1,4 +1,8 @@
 <?xml version="1.0"?>
 <robot>
+    <!-- Add color to the camera box -->
+    <gazebo reference="camera_link">
+        <material>Gazebo/Red</material>
+    </gazebo>
     <!-- Add a camera into Gazebo and a plugin to communicate its frames to ROS -->
     <gazebo reference="camera_link">

File: mobile_platform/platform_description/urdf/gazebo.xacro (robot description, xacro)
@@ -5,10 +5,10 @@
         <gravity>0</gravity>
     </gazebo>
-    <!-- <gazebo reference="base_roll_link">
+    <gazebo reference="base_roll_link">
         <gravity>0</gravity>
     </gazebo>
     <gazebo reference="base_pitch_link">
         <gravity>0</gravity>
-    </gazebo> -->
+    </gazebo>
     <!-- <gazebo reference="base_yaw_link">
         <gravity>0</gravity>

File: mobile_platform/platform_description/urdf/mobile_platform.xacro (robot description, xacro)
@@ -24,5 +24,5 @@
             <!-- Physical properties -->
             <xacro:if value="${inertial}">
-                <xacro:box_inertial x="${length}" y="${width}" z="${height}" mass="1"/>
+                <xacro:box_inertial x="${length}" y="${width}" z="${height}" mass="0.1"/>
             </xacro:if>
         </link>
@@ -35,5 +35,5 @@
             <origin xyz="${origin}"/>
             <axis xyz="${axis}"/>
-            <limit upper="1.57" lower="-1.57" effort="1" velocity="0.1"/>
+            <limit upper="1.57" lower="-1.57" effort="1" velocity="10"/>
             <!-- <dynamics damping="0.1" friction="0.1"/> -->
         </joint>
