Commit message: Camera working with rqt/image view

File: camera/urdf/camera.xacro (robot description, xacro)
@@ -4,5 +4,4 @@
     <xacro:include filename="camera_gazebo.xacro"/>
     <xacro:include filename="../../mobile_platform/platform_description/urdf/materials.xacro"/>
-    <!-- <xacro:include filename="world_link.xacro"/> -->
     <!-- Define a property to indicate the size of the camera box -->
     <xacro:property name="camera_size" value="0.1"/>

File: mobile_platform/platform_description/urdf/gazebo.xacro (robot description, xacro)
@@ -2,22 +2,19 @@
 <robot>
     <!-- Disable gravity for the platform -->
-    <gazebo reference="board_sup_link">
+    <gazebo reference="board_link">
         <gravity>0</gravity>
     </gazebo>
-    <!-- <gazebo reference="base1_link">
+    <!-- <gazebo reference="base_roll_link">
         <gravity>0</gravity>
     </gazebo>
-    <gazebo reference="base2_link">
+    <gazebo reference="base_pitch_link">
+        <gravity>0</gravity>
+    </gazebo> -->
+    <!-- <gazebo reference="base_yaw_link">
         <gravity>0</gravity>
     </gazebo> -->
     <!-- Add texture/colors to links -->
-    <gazebo reference="board_sup_link">
+    <gazebo reference="board_link">
         <material>PlatformPattern</material>
-    </gazebo>
-    <!-- <gazebo reference="board_sup_link">
-        <material>Gazebo/Red</material>
-    </gazebo> -->
-    <gazebo reference="board_inf_link">
-        <material>Gazebo/Green</material>
     </gazebo>
     <!-- ros_control model plugin -->

File: mobile_platform/platform_description/urdf/mobile_platform.xacro (robot description, xacro)
@@ -71,5 +71,4 @@
     <xacro:revolute_joint name="pitch" parent_name="base_pitch" child_name="base_roll" origin="0 0 0" axis="0 1 0"/>
     <xacro:revolute_joint name="roll" parent_name="base_roll" child_name="board" origin="0 0 0" axis="1 0 0"/>
-    <!-- FIXME: -->
     <!-- Transmissions -->
     <!-- FIXME: -->

Commit message: Implemented an error function

File: camera/urdf/camera.xacro (robot description, xacro)
@@ -36,4 +36,5 @@
         <parent link="world"/>
         <child link="camera_link"/>
+        <origin xyz ="0 0 2.5" rpy="0 1.57079632679 0"/>
     </joint>
 </robot>

File: mobile_platform/platform_description/urdf/mobile_platform.xacro (robot description, xacro)
@@ -65,4 +65,5 @@
         <parent link="world"/>
         <child link="base_yaw_link"/>
+        <origin xyz="0 0 1"/>
     </joint>
     <xacro:revolute_joint name="yaw" parent_name="base_yaw" child_name="base_pitch" origin="0 0 0" axis="0 0 1"/>

Commit message: Fixed some issues (delayed the position command, marked the pose_topic as latch,...)

File: camera/urdf/camera.xacro (robot description, xacro)
@@ -19,4 +19,7 @@
                 <box size="${camera_size} ${camera_size} ${camera_size}"/>
             </geometry>
+            <!-- <geometry>
+                <mesh filename="../meshes/test.stl" scale="0.001 0.001 0.001"/>
+            </geometry> -->
             <material name="red"/>
         </visual>
@@ -25,4 +28,7 @@
                 <box size="${camera_size} ${camera_size} ${camera_size}"/>
             </geometry>
+            <!-- <geometry>
+                <mesh filename="file://media/tom/Shared/Stage-EN-2022/quadcopter_landing_ws/src/camera/meshes/STD04_0000_Hexapode-MISTRAL_600.stl" scale="0.001 0.001 0.001"/>
+            </geometry> -->
         </collision>
         <inertial>

File: camera/urdf/depth_camera_gazebo.xacro (robot description, xacro)
@@ -9,5 +9,5 @@
         <sensor name="camera1" type="depth">
             <always_on>true</always_on>
-            <update_rate>30.0</update_rate>
+            <update_rate>50.0</update_rate>
             <camera>
                 <horizontal_fov>1.3962634</horizontal_fov>
@@ -24,5 +24,5 @@
                     <type>gaussian</type>
                     <mean>0.0</mean>
-                    <stddev>0.007</stddev>
+                    <stddev>0.0</stddev>
                 </noise>
             </camera>

File: mobile_platform/platform_description/urdf/mobile_platform.xacro (robot description, xacro)
@@ -65,5 +65,5 @@
         <parent link="world"/>
         <child link="base_yaw_link"/>
-        <origin xyz="0 0 1"/>
+        <origin xyz="0 0 1."/>
     </joint>
     <xacro:revolute_joint name="yaw" parent_name="base_yaw" child_name="base_pitch" origin="0 0 0" axis="0 0 1"/>

Commit message: Implemented a pose estimation procedure based on blind PnP

File: camera/urdf/camera.xacro (robot description, xacro)
@@ -18,4 +18,5 @@
             <geometry>
                 <box size="${camera_size} ${camera_size} ${camera_size}"/>
+                <!-- <mesh filename="../meshes/Hexa.obj" scale="0.001 0.001 0.001"/> -->
             </geometry>
             <!-- <geometry>
@@ -27,4 +28,5 @@
             <geometry>
                 <box size="${camera_size} ${camera_size} ${camera_size}"/>
+                <!-- <mesh filename="../meshes/Hexa.obj" scale="0.001 0.001 0.001"/> -->
             </geometry>
             <!-- <geometry>

File: mobile_platform/platform_description/urdf/gazebo.xacro (robot description, xacro)
@@ -14,5 +14,4 @@
         <gravity>0</gravity>
     </gazebo>
-    <!-- TODO: -->
     <gazebo reference="base_tx_link">
         <gravity>0</gravity>

File: mobile_platform/platform_description/urdf/mobile_platform.xacro (robot description, xacro)
@@ -39,5 +39,4 @@
         </joint>
     </xacro:macro>
-    <!-- TODO: Gather revolute and prismatic joints in a single macro-->
     <!-- Simple prismatic joint -->
     <xacro:macro name="prismatic_joint" params="name parent_name child_name origin axis">

Commit message: Added an Iris drone model to the simulation and a MAVROS launcher to allow us controlling it with ROS

File: camera/urdf/camera.xacro (robot description, xacro)
@@ -28,5 +28,4 @@
             <geometry>
                 <box size="${camera_size} ${camera_size} ${camera_size}"/>
-                <!-- <mesh filename="../meshes/Hexa.obj" scale="0.001 0.001 0.001"/> -->
             </geometry>
             <!-- <geometry>
