Commit message: Written a launch file to start a joint controller, joint position control working, workspace needs to be cleaned

File: mobile_platform/platform_description/urdf/gazebo.xacro (robot description, xacro)
@@ -3,22 +3,7 @@
     <!-- Add texture to the board -->
 <!-- A verifier -->
-    <gazebo reference="board">
+    <!-- <gazebo reference="board">
         <material>../materials/scripts/PlatformPattern</material>
-    </gazebo>
-    <!-- Transmission tags to actuate the platform -->
-    <!-- It links an actuator to a joint -->
-    <xacro:macro name="transmission" params="joint_name">
-        <transmission name="${joint_name}_transmission">
-            <type>transmission_interface/SimpleTransmission</type>
-            <joint name="${joint_name}_joint">
-                <!-- We can change the hardware interface to control position, velocity or effort -->
-                <hardwareInterface>hardware_interface/PositionJointInterface</hardwareInterface>
-            </joint>
-            <actuator name="${joint_name}_actuator">
-                <hardwareInterface>hardware_interface/PositionJointInterface</hardwareInterface>
-                <mechanicalReduction>1</mechanicalReduction>
-            </actuator>
-        </transmission>
-    </xacro:macro>
+    </gazebo> -->
     <!-- ros_control plugin -->
     <gazebo>

File: mobile_platform/platform_description/urdf/mobile_platform.xacro (robot description, xacro)
@@ -2,10 +2,11 @@
 <robot xmlns:xacro="http://www.ros.org/wiki/xacro" name="mobile_platform">
     <!--Include files-->
-    <!-- <xacro:include filename="gazebo.xacro" /> -->
+    <xacro:include filename="gazebo.xacro" />
     <xacro:include filename="inertias.xacro" />
     <xacro:include filename="materials.xacro" />
     <!--Define properties-->
     <!-- <xacro:property name="width" value="1" /> -->
-    <!--Define macros-->
+    <!--MACROS-->
+    <!-- Simple box link  -->
     <xacro:macro name="box_link" params="name length width height material inertial:=true">
         <link name="${name}_link">
@@ -27,6 +28,7 @@
         </link>
     </xacro:macro>
+    <!-- Simple revolute joint -->
     <xacro:macro name="revolute_joint" params="name parent_name child_name origin axis">
-        <joint name="${name}_revolute_joint" type="revolute">
+        <joint name="${name}_joint" type="revolute">
             <parent link="${parent_name}_link"/>
             <child link="${child_name}_link"/>
@@ -37,7 +39,24 @@
         </joint>
     </xacro:macro>
+    <!-- Transmission tags to actuate the platform -->
+    <!-- It links an actuator to a joint -->
+    <xacro:macro name="transmission" params="joint_name">
+        <transmission name="${joint_name}_transmission">
+            <type>transmission_interface/SimpleTransmission</type>
+            <joint name="${joint_name}_joint">
+                <!-- We can change the hardware interface to control position, velocity or effort -->
+                <hardwareInterface>hardware_interface/PositionJointInterface</hardwareInterface>
+            </joint>
+            <actuator name="${joint_name}_actuator">
+                <hardwareInterface>hardware_interface/PositionJointInterface</hardwareInterface>
+                <mechanicalReduction>1</mechanicalReduction>
+            </actuator>
+        </transmission>
+    </xacro:macro>
     <!-- Robot description -->
+    <!-- Links -->
     <xacro:box_link name="ground" length="0.1" width="0.1" height="0.1" material="green"/>
     <xacro:box_link name="board" length="1" width="1" height="0.05" material="red"/>
+    <!-- Joints -->
     <!-- <joint name="fixed" type="fixed">
         <parent link="world"/>
@@ -45,3 +64,5 @@
     </joint> -->
     <xacro:revolute_joint name="roll" parent_name="ground" child_name="board" origin="0 0 1" axis="1 0 0"/>
+    <!-- Transmissions -->
+    <xacro:transmission joint_name="roll"/>
 </robot>

Commit message: Fixed platform to the world and added texture

File: mobile_platform/platform_description/urdf/gazebo.xacro (robot description, xacro)
@@ -1,8 +1,10 @@
 <?xml version="1.0"?>
 <robot>
-    <!-- Add texture to the board -->
-<!-- A verifier -->
-    <!-- <gazebo reference="board">
-        <material>../materials/scripts/PlatformPattern</material>
+    <!-- Add texture/colors to links -->
+    <gazebo reference="board_link">
+        <material>PlatformPattern</material>
+    </gazebo>
+    <!-- <gazebo reference="board_link">
+        <material>Gazebo/Red</material>
     </gazebo> -->
     <!-- ros_control plugin -->

File: mobile_platform/platform_description/urdf/mobile_platform.xacro (robot description, xacro)
@@ -56,5 +56,6 @@
     <!-- Robot description -->
     <!-- Links -->
-    <xacro:box_link name="ground" length="0.1" width="0.1" height="0.1" material="green"/>
+    <link name="world_link"/>
+    <xacro:box_link name="base" length="0.1" width="0.1" height="0.1" material="green"/>
     <xacro:box_link name="board" length="1" width="1" height="0.05" material="red"/>
     <!-- Joints -->
@@ -63,5 +64,10 @@
         <child link="ground"/>
     </joint> -->
-    <xacro:revolute_joint name="roll" parent_name="ground" child_name="board" origin="0 0 1" axis="1 0 0"/>
+    <joint name="fixed" type="fixed">
+        <origin xyz="0 0 0" rpy="0 0 0" />
+        <parent link="world_link"/>
+        <child link="base_link"/>
+    </joint>
+    <xacro:revolute_joint name="roll" parent_name="base" child_name="board" origin="0 0 1" axis="1 0 0"/>
     <!-- Transmissions -->
     <xacro:transmission joint_name="roll"/>

Commit message: Removed gravity for the board and some physics properties, rviz working

File: mobile_platform/platform_description/urdf/gazebo.xacro (robot description, xacro)
@@ -1,4 +1,11 @@
 <?xml version="1.0"?>
 <robot>
+    <!-- Disable gravity for the platform -->
+    <gazebo reference="board_link">
+        <gravity>0</gravity>
+    </gazebo>
+    <!-- <gazebo reference="base_link">
+        <gravity>0</gravity>
+    </gazebo> -->
     <!-- Add texture/colors to links -->
     <gazebo reference="board_link">

File: mobile_platform/platform_description/urdf/mobile_platform.xacro (robot description, xacro)
@@ -36,5 +36,5 @@
             <axis xyz="${axis}"/>
             <limit upper="1.57" lower="-1.57" effort="1" velocity="0.1"/>
-            <dynamics damping="0.1" friction="0.1"/>
+            <!-- <dynamics damping="0.1" friction="0.1"/> -->
         </joint>
     </xacro:macro>
@@ -60,8 +60,4 @@
     <xacro:box_link name="board" length="1" width="1" height="0.05" material="red"/>
     <!-- Joints -->
-    <!-- <joint name="fixed" type="fixed">
-        <parent link="world"/>
-        <child link="ground"/>
-    </joint> -->
     <joint name="fixed" type="fixed">
         <origin xyz="0 0 0" rpy="0 0 0" />

Commit message: Cut the board in two links and added a fixed joint between them

File: mobile_platform/platform_description/urdf/gazebo.xacro (robot description, xacro)
@@ -2,5 +2,8 @@
 <robot>
     <!-- Disable gravity for the platform -->
-    <gazebo reference="board_link">
+    <gazebo reference="board_sup_link">
+        <gravity>0</gravity>
+    </gazebo>
+    <gazebo reference="board_inf_link">
         <gravity>0</gravity>
     </gazebo>
@@ -8,11 +11,15 @@
         <gravity>0</gravity>
     </gazebo> -->
+    <!-- FIXME: -->
     <!-- Add texture/colors to links -->
-    <gazebo reference="board_link">
+    <gazebo reference="board_sup_link">
         <material>PlatformPattern</material>
     </gazebo>
-    <!-- <gazebo reference="board_link">
+    <!-- <gazebo reference="board_sup_link">
         <material>Gazebo/Red</material>
     </gazebo> -->
+    <gazebo reference="board_inf_link">
+        <material>Gazebo/Green</material>
+    </gazebo>
     <!-- ros_control plugin -->
     <gazebo>

File: mobile_platform/platform_description/urdf/mobile_platform.xacro (robot description, xacro)
@@ -58,5 +58,7 @@
     <link name="world_link"/>
     <xacro:box_link name="base" length="0.1" width="0.1" height="0.1" material="green"/>
-    <xacro:box_link name="board" length="1" width="1" height="0.05" material="red"/>
+    <!-- FIXME: -->
+    <xacro:box_link name="board_sup" length="1" width="1" height="0.05" material="red"/>
+    <xacro:box_link name="board_inf" length="1" width="1" height="0.05" material="red"/>
     <!-- Joints -->
     <joint name="fixed" type="fixed">
@@ -65,6 +67,16 @@
         <child link="base_link"/>
     </joint>
-    <xacro:revolute_joint name="roll" parent_name="base" child_name="board" origin="0 0 1" axis="1 0 0"/>
+    <!-- FIXME: -->
+    <xacro:revolute_joint name="roll" parent_name="base" child_name="board_sup" origin="0 0 1" axis="1 0 0"/>
+    <xacro:revolute_joint name="pitch" parent_name="base" child_name="board_inf" origin="0 0 1" axis="0 1 0"/>
+    <gazebo>
+        <joint name="fixed_board" type="fixed">
+            <parent>board_sup_link</parent>
+            <child>board_inf_link</child>
+        </joint>
+    </gazebo>
     <!-- Transmissions -->
+    <!-- FIXME: -->
     <xacro:transmission joint_name="roll"/>
+    <xacro:transmission joint_name="pitch"/>
 </robot>

Commit message: First try with two serial rotations

File: mobile_platform/platform_description/urdf/gazebo.xacro (robot description, xacro)
@@ -3,4 +3,7 @@
     <!-- Disable gravity for the platform -->
     <gazebo reference="board_link">
+        <gravity>0</gravity>
+    </gazebo>
+    <gazebo reference="base2_link">
         <gravity>0</gravity>
     </gazebo>

File: mobile_platform/platform_description/urdf/mobile_platform.xacro (robot description, xacro)
@@ -57,15 +57,20 @@
     <!-- Links -->
     <link name="world_link"/>
-    <xacro:box_link name="base" length="0.1" width="0.1" height="0.1" material="green"/>
+    <!-- FIXME: -->
+    <xacro:box_link name="base1" length="0.1" width="0.1" height="0.1" material="green"/>
+    <xacro:box_link name="base2" length="0.1" width="0.1" height="0.1" material="green"/>
     <xacro:box_link name="board" length="1" width="1" height="0.05" material="red"/>
     <!-- Joints -->
+    <!-- FIXME: -->
     <joint name="fixed" type="fixed">
         <origin xyz="0 0 0" rpy="0 0 0" />
         <parent link="world_link"/>
-        <child link="base_link"/>
+        <child link="base1_link"/>
     </joint>
-    <xacro:revolute_joint name="roll" parent_name="base" child_name="board" origin="0 0 1" axis="1 0 0"/>
+    <xacro:revolute_joint name="pitch" parent_name="base1" child_name="base2" origin="0 0 1" axis="0 1 0"/>
+    <xacro:revolute_joint name="roll" parent_name="base2" child_name="board" origin="0 0 1" axis="1 0 0"/>
+    <!-- FIXME: -->
     <!-- Transmissions -->
     <xacro:transmission joint_name="roll"/>
-<!-- blabla -->
+    <xacro:transmission joint_name="pitch"/>
 </robot>

Commit message: Added pitch and yaw rotations

File: mobile_platform/platform_description/urdf/gazebo.xacro (robot description, xacro)
@@ -5,8 +5,8 @@
         <gravity>0</gravity>
     </gazebo>
-    <gazebo reference="base2_link">
+    <!-- <gazebo reference="base1_link">
         <gravity>0</gravity>
     </gazebo>
-    <!-- <gazebo reference="base_link">
+    <gazebo reference="base2_link">
         <gravity>0</gravity>
     </gazebo> -->

File: mobile_platform/platform_description/urdf/mobile_platform.xacro (robot description, xacro)
@@ -56,21 +56,23 @@
     <!-- Robot description -->
     <!-- Links -->
-    <link name="world_link"/>
+    <link name="world"/>
     <!-- FIXME: -->
-    <xacro:box_link name="base1" length="0.1" width="0.1" height="0.1" material="green"/>
-    <xacro:box_link name="base2" length="0.1" width="0.1" height="0.1" material="green"/>
-    <xacro:box_link name="board" length="1" width="1" height="0.05" material="red"/>
+    <xacro:box_link name="base_yaw" length="0" width="0" height="0" material="red"/>
+    <xacro:box_link name="base_pitch" length="0" width="0" height="0" material="red"/>
+    <xacro:box_link name="base_roll" length="0" width="0" height="0" material="red"/>
+    <xacro:box_link name="board" length="1" width="1" height="0.05" material="green"/>
     <!-- Joints -->
     <!-- FIXME: -->
     <joint name="fixed" type="fixed">
-        <origin xyz="0 0 0" rpy="0 0 0" />
-        <parent link="world_link"/>
-        <child link="base1_link"/>
+        <parent link="world"/>
+        <child link="base_yaw_link"/>
     </joint>
-    <xacro:revolute_joint name="pitch" parent_name="base1" child_name="base2" origin="0 0 1" axis="0 1 0"/>
-    <xacro:revolute_joint name="roll" parent_name="base2" child_name="board" origin="0 0 1" axis="1 0 0"/>
+    <xacro:revolute_joint name="yaw" parent_name="base_yaw" child_name="base_pitch" origin="0 0 0" axis="0 0 1"/>
+    <xacro:revolute_joint name="pitch" parent_name="base_pitch" child_name="base_roll" origin="0 0 0" axis="0 1 0"/>
+    <xacro:revolute_joint name="roll" parent_name="base_roll" child_name="board" origin="0 0 0" axis="1 0 0"/>
     <!-- FIXME: -->
     <!-- Transmissions -->
     <xacro:transmission joint_name="roll"/>
     <xacro:transmission joint_name="pitch"/>
+    <xacro:transmission joint_name="yaw"/>
 </robot>

Commit message: Added the 3 translations and implemented a service to reset simultaneously all joints values

File: mobile_platform/platform_description/urdf/gazebo.xacro (robot description, xacro)
@@ -11,7 +11,17 @@
         <gravity>0</gravity>
     </gazebo>
-    <!-- <gazebo reference="base_yaw_link">
+    <gazebo reference="base_yaw_link">
         <gravity>0</gravity>
-    </gazebo> -->
+    </gazebo>
+    <!-- TODO: -->
+    <gazebo reference="base_tx_link">
+        <gravity>0</gravity>
+    </gazebo>
+    <gazebo reference="base_ty_link">
+        <gravity>0</gravity>
+    </gazebo>
+    <gazebo reference="base_tz_link">
+        <gravity>0</gravity>
+    </gazebo>
     <!-- Add texture/colors to links -->
     <gazebo reference="board_link">

File: mobile_platform/platform_description/urdf/mobile_platform.xacro (robot description, xacro)
@@ -35,6 +35,18 @@
             <origin xyz="${origin}"/>
             <axis xyz="${axis}"/>
-            <limit upper="1.57" lower="-1.57" effort="1" velocity="10"/>
-            <!-- <dynamics damping="0.1" friction="0.1"/> -->
+            <limit upper="1.57" lower="-1.57" effort="5" velocity="10"/>
+            <dynamics damping="0.1" friction="0.1"/>
+        </joint>
+    </xacro:macro>
+    <!-- TODO: Gather revolute and prismatic joints in a single macro-->
+    <!-- Simple prismatic joint -->
+    <xacro:macro name="prismatic_joint" params="name parent_name child_name origin axis">
+        <joint name="${name}_joint" type="prismatic">
+            <parent link="${parent_name}_link"/>
+            <child link="${child_name}_link"/>
+            <origin xyz="${origin}"/>
+            <axis xyz="${axis}"/>
+            <limit upper="3.0" lower="-3.0" effort="5" velocity="10"/>
+            <dynamics damping="0.1" friction="0.1"/>
         </joint>
     </xacro:macro>
@@ -57,4 +69,7 @@
     <!-- Links -->
     <link name="world"/>
+    <xacro:box_link name="base_tx" length="0" width="0" height="0" material="red"/>
+    <xacro:box_link name="base_ty" length="0" width="0" height="0" material="red"/>
+    <xacro:box_link name="base_tz" length="0" width="0" height="0" material="red"/>
     <xacro:box_link name="base_yaw" length="0" width="0" height="0" material="red"/>
     <xacro:box_link name="base_pitch" length="0" width="0" height="0" material="red"/>
@@ -64,11 +79,17 @@
     <joint name="fixed" type="fixed">
         <parent link="world"/>
-        <child link="base_yaw_link"/>
+        <child link="base_tx_link"/>
         <origin xyz="0 0 1."/>
     </joint>
+    <xacro:prismatic_joint name="tx" parent_name="base_tx" child_name="base_ty" origin="0 0 0" axis="1 0 0"/>
+    <xacro:prismatic_joint name="ty" parent_name="base_ty" child_name="base_tz" origin="0 0 0" axis="0 1 0"/>
+    <xacro:prismatic_joint name="tz" parent_name="base_tz" child_name="base_yaw" origin="0 0 0" axis="0 0 1"/>
     <xacro:revolute_joint name="yaw" parent_name="base_yaw" child_name="base_pitch" origin="0 0 0" axis="0 0 1"/>
     <xacro:revolute_joint name="pitch" parent_name="base_pitch" child_name="base_roll" origin="0 0 0" axis="0 1 0"/>
     <xacro:revolute_joint name="roll" parent_name="base_roll" child_name="board" origin="0 0 0" axis="1 0 0"/>
     <!-- Transmissions -->
+    <xacro:transmission joint_name="tx"/>
+    <xacro:transmission joint_name="ty"/>
+    <xacro:transmission joint_name="tz"/>
     <xacro:transmission joint_name="roll"/>
     <xacro:transmission joint_name="pitch"/>
