Commit message: Synchronized the sinusoid and cleaned the code

File: mobile_platform/platform_description/urdf/mobile_platform.xacro (robot description, xacro)
@@ -65,5 +65,5 @@
         <parent link="world"/>
         <child link="base_yaw_link"/>
-        <origin xyz="0 0 1"/>
+        <origin xyz="0 0 1.5"/>
     </joint>
     <xacro:revolute_joint name="yaw" parent_name="base_yaw" child_name="base_pitch" origin="0 0 0" axis="0 0 1"/>

Commit message: Fixed the axes' issue

File: mobile_platform/platform_description/urdf/mobile_platform.xacro (robot description, xacro)
@@ -65,5 +65,5 @@
         <parent link="world"/>
         <child link="base_yaw_link"/>
-        <origin xyz="0 0 1.5"/>
+        <origin xyz="0 0 1"/>
     </joint>
     <xacro:revolute_joint name="yaw" parent_name="base_yaw" child_name="base_pitch" origin="0 0 0" axis="0 0 1"/>

Commit message: Used an action to stabilize the drone and a state machine to structure the entire landing procedure

File: mobile_platform/platform_description/urdf/mobile_platform.xacro (robot description, xacro)
@@ -35,6 +35,6 @@
             <origin xyz="${origin}"/>
             <axis xyz="${axis}"/>
-            <limit upper="1.57" lower="-1.57" effort="5" velocity="10"/>
-            <dynamics damping="0.1" friction="0.1"/>
+            <limit upper="1.57" lower="-1.57" effort="500" velocity="10"/>
+            <dynamics damping="0.1" friction="100"/>
         </joint>
     </xacro:macro>
@@ -46,6 +46,6 @@
             <origin xyz="${origin}"/>
             <axis xyz="${axis}"/>
-            <limit upper="3.0" lower="-3.0" effort="5" velocity="10"/>
-            <dynamics damping="0.1" friction="0.1"/>
+            <limit upper="3.0" lower="-3.0" effort="500" velocity="10"/>
+            <dynamics damping="0.1" friction="100"/>
         </joint>
     </xacro:macro>

Commit message: Added pose estimation and landing decision actions, used a concurrence container in the state machine and started working on predictive decisionning

File: mobile_platform/platform_description/urdf/mobile_platform.xacro (robot description, xacro)
@@ -36,5 +36,5 @@
             <axis xyz="${axis}"/>
             <limit upper="1.57" lower="-1.57" effort="500" velocity="10"/>
-            <dynamics damping="0.1" friction="100"/>
+            <dynamics damping="0.1" friction="0.1"/>
         </joint>
     </xacro:macro>
@@ -47,5 +47,5 @@
             <axis xyz="${axis}"/>
             <limit upper="3.0" lower="-3.0" effort="500" velocity="10"/>
-            <dynamics damping="0.1" friction="100"/>
+            <dynamics damping="0.1" friction="0.1"/>
         </joint>
     </xacro:macro>
